File: octalPointsense/octalPointsense.kicad_pcb (KiCad board)
At the start: 2 copper layers, 44.5 x 82.6 mm, 20 parts, among them J101 Turnout 2, J102 Turnout 1, J103 To Tower, J104 Turnout 3, J105 Turnout 4, J106 Turnout 5, J107 Turnout 6, J108 Turnout 7, J109 Turnout 8, U101 74HC00, U102 74HC00, U103 74HC00, U104 74HC00

Commit message: Replace 74ht00 with 74ht03 (open drain) and add 1K series resistors.
Parts:
- added R101: 1K, Resistor_SMD:R_0603_1608Metric, F.Cu at (75.4, 67.6)
- added R102: 1K, Resistor_SMD:R_0603_1608Metric, F.Cu at (72.9, 69.2)
- added R103: 1K, Resistor_SMD:R_0603_1608Metric, F.Cu at (78.2, 84.6)
- added R104: 1K, Resistor_SMD:R_0603_1608Metric, F.Cu at (78.0, 86.9)
- added R105: 1K, Resistor_SMD:R_0603_1608Metric, F.Cu at (69.8, 100.0)
- added R106: 1K, Resistor_SMD:R_0603_1608Metric, F.Cu at (78.2, 93.0)
- added R107: 1K, Resistor_SMD:R_0603_1608Metric, F.Cu at (72.4, 100.3)
- added R108: 1K, Resistor_SMD:R_0603_1608Metric, F.Cu at (74.9, 100.3)
- U101, U102, U103, U104: value 74HC00 -> 74HC03
Connections:
- U101 pad 12: /Line 2 -> Net-(U101-Pad12)
- U101 pad 3: /Line 1 -> Net-(U101-Pad3)
- U101 pad 4: /Line 1 -> Net-(U101-Pad3)
- U101 pad 8: /Line 2 -> Net-(U101-Pad12)
- U102 pad 12: /Line 4 -> Net-(U102-Pad12)
- U102 pad 3: /Line 3 -> Net-(U102-Pad3)
- U102 pad 4: /Line 3 -> Net-(U102-Pad3)
- U102 pad 8: /Line 4 -> Net-(U102-Pad12)
- U103 pad 12: /Line 6 -> Net-(U103-Pad12)
- U103 pad 3: /Line 5 -> Net-(U103-Pad3)
- U103 pad 4: /Line 5 -> Net-(U103-Pad3)
- U103 pad 8: /Line 6 -> Net-(U103-Pad12)
- U104 pad 12: /Line 8 -> Net-(U104-Pad8)
- U104 pad 3: /Line 7 -> Net-(U104-Pad3)
- U104 pad 4: /Line 7 -> Net-(U104-Pad3)
- U104 pad 8: /Line 8 -> Net-(U104-Pad8)
Routing:
- net /Line 8: track 54.6 -> 4.15 mm, vias 2 -> 0
- net Net-(U104-Pad8): track 0.00 -> 48.5 mm, vias 0 -> 2
- net /Line 7: track 43.2 -> 4.15 mm, vias 2 -> 0
- net Net-(U104-Pad3): track 0.00 -> 37.6 mm, vias 0 -> 2
- net /Line 6: track 35.4 -> 2.92 mm, vias 1 -> 0
- net Net-(U103-Pad12): track 0.00 -> 30.8 mm, vias 0 -> 2
- net /Line 2: track 44.3 -> 17.4 mm, vias 2 -> 0
- net /Line 1: track 41.1 -> 15.8 mm, vias 2 -> 0
- net Net-(U101-Pad12): track 0.00 -> 25.3 mm, vias 0 -> 2
- net Net-(U101-Pad3): track 0.00 -> 23.6 mm, vias 0 -> 2
- net /Line 5: track 30.6 -> 7.07 mm, vias 2 -> 0
- net Net-(U103-Pad3): track 0.00 -> 21.9 mm, vias 0 -> 2
- net /Line 4: track 25.0 -> 3.15 mm, vias 1 -> 0
- net Net-(U102-Pad12): track 0.00 -> 20.2 mm, vias 0 -> 2
- net /Line 3: track 19.0 -> 6.89 mm, vias 1 -> 0
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