File: octalPointsense/octalPointsense.kicad_sch (KiCad schematic)
At the start: 20 parts, among them J101 Turnout 2, J102 Turnout 1, J103 To Tower, J104 Turnout 3, J105 Turnout 4, J106 Turnout 5, J107 Turnout 6, J108 Turnout 7, J109 Turnout 8, U101 74HC00, U102 74HC00, U103 74HC00, U104 74HC00

Commit message: Replace 74ht00 with 74ht03 (open drain) and add 1K series resistors.
Parts:
- added R101, R102, R103, R104, R105, R106, R107, R108: 1K, Resistor_SMD:R_0603_1608Metric, symbol Device:R
- U101, U102, U103, U104: value 74HC00 -> 74HC03; Manufacturer Diodes Incorporated -> Nexperia; Manufacturer Part Number 74HCT00T14-13 -> 74HC03PW,118; Mouser Part Number 621-74HCT00T14-13 -> 771-HC03PW118
- U101: value 74HC00 -> 74HC03; Manufacturer Diodes Incorporated -> Nexperia; Mouser Part Number 621-74HCT00T14-13 -> 771-HC03PW118
Connections:
- net Line 1: now also R102.1; no longer U101.3, U101.4
- net Line 2: now also R101.1; no longer U101.12, U101.8
- net Line 3: now also R103.1; no longer U102.3, U102.4
- net Line 4: now also R104.1; no longer U102.12, U102.8
- net Line 5: now also R105.1; no longer U103.3, U103.4
- net Line 6: now also R106.1; no longer U103.12, U103.8
- net Line 7: now also R107.1; no longer U104.3, U104.4
- net Line 8: now also R108.1; no longer U104.12, U104.8
- new net: R102.2, U101.3, U101.4
- new net: R101.2, U101.12, U101.8
- new net: R103.2, U102.3, U102.4
- new net: R104.2, U102.12, U102.8
- new net: R107.2, U104.3, U104.4
- new net: R105.2, U103.3, U103.4
- new net: R108.2, U104.12, U104.8
- new net: R106.2, U103.12, U103.8
